Commit message: Updated urdf

File: urdf/arm_main.xacro (robot description, xacro)
@@ -5,7 +5,7 @@
 <link name="base_link">
   <inertial>
-    <origin xyz="-0.0012214089016151053 0.02712127606702909 -0.02444560560426352" rpy="0 0 0"/>
-    <mass value="0.8833573620888653"/>
-    <inertia ixx="0.001118" iyy="0.000472" izz="0.000805" ixy="3e-06" iyz="0.000355" ixz="-4e-06"/>
+    <origin xyz="-0.0013499999845841886 0.05547364405613593 -0.03925880078129778" rpy="0 0 0"/>
+    <mass value="0.3900830776668987"/>
+    <inertia ixx="0.000131" iyy="7.1e-05" izz="0.000111" ixy="-0.0" iyz="2e-06" ixz="0.0"/>
   </inertial>
   <visual>
@@ -23,107 +23,133 @@
   </collision>
 </link>
-<link name="servo_holder2_v2_1">
+<link name="servo_holder2_v9_1">
   <inertial>
-    <origin xyz="-0.023124515666649855 0.08470253666904037 -8.411334129210246e-12" rpy="0 0 0"/>
-    <mass value="0.7144775958239902"/>
-    <inertia ixx="0.001083" iyy="0.000178" izz="0.001183" ixy="-2e-06" iyz="0.0" ixz="0.0"/>
+    <origin xyz="-0.022087999236917965 -0.042450935490717844 1.2480391720082196e-11" rpy="0 0 0"/>
+    <mass value="0.4815312282713089"/>
+    <inertia ixx="0.000189" iyy="0.000107" izz="0.000233" ixy="1e-06" iyz="-0.0" ixz="-0.0"/>
   </inertial>
   <visual>
-    <origin xyz="-0.0227 -0.1264 -0.04195" rpy="0 0 0"/>
+    <origin xyz="-0.0217 -0.0324 -0.04195" rpy="0 0 0"/>
     <geometry>
-      <mesh filename="package://arm_main_description/meshes/servo_holder2_v2_1.stl" scale="0.001 0.001 0.001"/>
+      <mesh filename="package://arm_main_description/meshes/servo_holder2_v9_1.stl" scale="0.001 0.001 0.001"/>
     </geometry>
     <material name="steel_satin"/>
   </visual>
   <collision>
-    <origin xyz="-0.0227 -0.1264 -0.04195" rpy="0 0 0"/>
+    <origin xyz="-0.0217 -0.0324 -0.04195" rpy="0 0 0"/>
     <geometry>
-      <mesh filename="package://arm_main_description/meshes/servo_holder2_v2_1.stl" scale="0.001 0.001 0.001"/>
+      <mesh filename="package://arm_main_description/meshes/servo_holder2_v9_1.stl" scale="0.001 0.001 0.001"/>
     </geometry>
   </collision>
 </link>
-<link name="hand_rotation_v11_4">
+<link name="hand_rotation_v13_4">
   <inertial>
-    <origin xyz="-0.023199999989499457 0.03605179829238042 -0.019122913280508146" rpy="0 0 0"/>
-    <mass value="0.5077046555158917"/>
-    <inertia ixx="0.000247" iyy="0.000181" izz="0.000228" ixy="-0.0" iyz="7e-06" ixz="0.0"/>
+    <origin xyz="-0.023199999989310653 -0.03180704370383808 0.018913049005446277" rpy="0 0 0"/>
+    <mass value="0.49875676728406393"/>
+    <inertia ixx="0.000221" iyy="0.000177" izz="0.0002" ixy="-0.0" iyz="7e-06" ixz="-0.0"/>
   </inertial>
   <visual>
-    <origin xyz="-0.0227 -0.2576 -0.04195" rpy="0 0 0"/>
+    <origin xyz="-0.0227 0.0338 -0.04195" rpy="0 0 0"/>
     <geometry>
-      <mesh filename="package://arm_main_description/meshes/hand_rotation_v11_4.stl" scale="0.001 0.001 0.001"/>
+      <mesh filename="package://arm_main_description/meshes/hand_rotation_v13_4.stl" scale="0.001 0.001 0.001"/>
     </geometry>
     <material name="steel_satin"/>
   </visual>
   <collision>
-    <origin xyz="-0.0227 -0.2576 -0.04195" rpy="0 0 0"/>
+    <origin xyz="-0.0227 0.0338 -0.04195" rpy="0 0 0"/>
     <geometry>
-      <mesh filename="package://arm_main_description/meshes/hand_rotation_v11_4.stl" scale="0.001 0.001 0.001"/>
+      <mesh filename="package://arm_main_description/meshes/hand_rotation_v13_4.stl" scale="0.001 0.001 0.001"/>
     </geometry>
   </collision>
 </link>
-<link name="hand_v15_1">
+<link name="hand_v17_1">
   <inertial>
-    <origin xyz="0.0018662468545444656 0.046209557945012414 -9.894154345851947e-06" rpy="0 0 0"/>
-    <mass value="0.8683719536760056"/>
-    <inertia ixx="0.000728" iyy="0.000758" izz="0.001224" ixy="0.000141" iyz="-2e-06" ixz="8e-06"/>
+    <origin xyz="0.0018876663935760566 -0.04171122715355233 1.0007712861637152e-05" rpy="0 0 0"/>
+    <mass value="0.8585184504197826"/>
+    <inertia ixx="0.000709" iyy="0.000757" izz="0.001205" ixy="-0.000142" iyz="-2e-06" ixz="-8e-06"/>
   </inertial>
   <visual>
-    <origin xyz="0.0005 -0.318 -0.04195" rpy="0 0 0"/>
+    <origin xyz="0.0005 0.0892 -0.04195" rpy="0 0 0"/>
     <geometry>
-      <mesh filename="package://arm_main_description/meshes/hand_v15_1.stl" scale="0.001 0.001 0.001"/>
+      <mesh filename="package://arm_main_description/meshes/hand_v17_1.stl" scale="0.001 0.001 0.001"/>
     </geometry>
     <material name="steel_satin"/>
   </visual>
   <collision>
-    <origin xyz="0.0005 -0.318 -0.04195" rpy="0 0 0"/>
+    <origin xyz="0.0005 0.0892 -0.04195" rpy="0 0 0"/>
     <geometry>
-      <mesh filename="package://arm_main_description/meshes/hand_v15_1.stl" scale="0.001 0.001 0.001"/>
+      <mesh filename="package://arm_main_description/meshes/hand_v17_1.stl" scale="0.001 0.001 0.001"/>
     </geometry>
   </collision>
 </link>
-<link name="servo_holder_v15_3">
+<link name="servo_holder_v23_3">
   <inertial>
-    <origin xyz="-0.02326241518713279 0.09672306724863754 0.006744967499623274" rpy="0 0 0"/>
-    <mass value="0.6761166227960398"/>
-    <inertia ixx="0.001236" iyy="0.000249" izz="0.001269" ixy="1e-06" iyz="-0.000135" ixz="1e-06"/>
+    <origin xyz="-0.021805779723410443 0.030701332587508144 0.01143066713838994" rpy="0 0 0"/>
+    <mass value="0.39894172696668956"/>
+    <inertia ixx="0.000121" iyy="0.000134" izz="9.8e-05" ixy="0.0" iyz="-8e-06" ixz="1e-06"/>
   </inertial>
   <visual>
-    <origin xyz="-0.0227 -0.0 -0.0125" rpy="0 0 0"/>
+    <origin xyz="-0.0212 -0.0 -0.0125" rpy="0 0 0"/>
     <geometry>
-      <mesh filename="package://arm_main_description/meshes/servo_holder_v15_3.stl" scale="0.001 0.001 0.001"/>
+      <mesh filename="package://arm_main_description/meshes/servo_holder_v23_3.stl" scale="0.001 0.001 0.001"/>
     </geometry>
     <material name="steel_satin"/>
   </visual>
   <collision>
-    <origin xyz="-0.0227 -0.0 -0.0125" rpy="0 0 0"/>
+    <origin xyz="-0.0212 -0.0 -0.0125" rpy="0 0 0"/>
     <geometry>
-      <mesh filename="package://arm_main_description/meshes/servo_holder_v15_3.stl" scale="0.001 0.001 0.001"/>
+      <mesh filename="package://arm_main_description/meshes/servo_holder_v23_3.stl" scale="0.001 0.001 0.001"/>
+    </geometry>
+  </collision>
+</link>
+<link name="base_mount_v2_1">
+  <inertial>
+    <origin xyz="0.00023028138914044723 -0.03219987847844947 0.0037687224019273234" rpy="0 0 0"/>
+    <mass value="0.4932742844219664"/>
+    <inertia ixx="0.000272" iyy="0.000248" izz="0.000132" ixy="1e-06" iyz="6e-05" ixz="-2e-06"/>
+  </inertial>
+  <visual>
+    <origin xyz="0.00135 -0.0369 0.0165" rpy="0 0 0"/>
+    <geometry>
+      <mesh filename="package://arm_main_description/meshes/base_mount_v2_1.stl" scale="0.001 0.001 0.001"/>
+    </geometry>
+    <material name="steel_satin"/>
+  </visual>
+  <collision>
+    <origin xyz="0.00135 -0.0369 0.0165" rpy="0 0 0"/>
+    <geometry>
+      <mesh filename="package://arm_main_description/meshes/base_mount_v2_1.stl" scale="0.001 0.001 0.001"/>
     </geometry>
   </collision>
 </link>
 <joint name="Revolute 7" type="continuous">
-  <origin xyz="0.0 0.1264 0.02945" rpy="0 0 0"/>
-  <parent link="servo_holder_v15_3"/>
-  <child link="servo_holder2_v2_1"/>
-  <axis xyz="-1.0 0.0 0.0"/>
+  <origin xyz="0.0005 0.0324 0.02945" rpy="0 0 0"/>
+  <parent link="servo_holder_v23_3"/>
+  <child link="servo_holder2_v9_1"/>
+  <axis xyz="1.0 -0.0 0.0"/>
 </joint>
 <joint name="Revolute 8" type="continuous">
-  <origin xyz="0.0 0.1312 0.0" rpy="0 0 0"/>
-  <parent link="servo_holder2_v2_1"/>
-  <child link="hand_rotation_v11_4"/>
-  <axis xyz="1.0 -0.0 -0.0"/>
+  <origin xyz="0.001 -0.0662 0.0" rpy="0 0 0"/>
+  <parent link="servo_holder2_v9_1"/>
+  <child link="hand_rotation_v13_4"/>
+  <axis xyz="1.0 0.0 0.0"/>
 </joint>
 <joint name="Revolute 9" type="continuous">
-  <origin xyz="-0.0232 0.0604 0.0" rpy="0 0 0"/>
-  <parent link="hand_rotation_v11_4"/>
-  <child link="hand_v15_1"/>
-  <axis xyz="-0.0 -1.0 -0.0"/>
+  <origin xyz="-0.0232 -0.0554 0.0" rpy="0 0 0"/>
+  <parent link="hand_rotation_v13_4"/>
+  <child link="hand_v17_1"/>
+  <axis xyz="-0.0 1.0 0.0"/>
 </joint>
 <joint name="Revolute 11" type="continuous">
-  <origin xyz="0.0227 0.0 0.0125" rpy="0 0 0"/>
-  <parent link="base_link"/>
-  <child link="servo_holder_v15_3"/>
+  <origin xyz="0.02255 -0.0369 0.029" rpy="0 0 0"/>
+  <parent link="base_mount_v2_1"/>
+  <child link="servo_holder_v23_3"/>
   <axis xyz="-1.0 -0.0 -0.0"/>
 </joint>
+<joint name="Revolute 12" type="continuous">
+  <origin xyz="-0.00135 0.0369 -0.0165" rpy="0 0 0"/>
+  <parent link="base_link"/>
+  <child link="base_mount_v2_1"/>
+  <axis xyz="0.0 -0.0 -1.0"/>
+</joint>
 </robot>

File: urdf/komarm.urdf (robot description, URDF)
Before this commit: robot arm_main, 5 links, 4 joints
Links:
- removed link hand_rotation_v11_4
- removed link hand_v15_1
- removed link servo_holder2_v2_1
- removed link servo_holder_v15_3
- added link base_mount_v2_1, mass 0.4932742844219664; collision mesh filename=../meshes/base_mount_v2_1.stl scale=0.001 0.001 0.001; visual mesh filename=../meshes/base_mount_v2_1.stl scale=0.001 0.001 0.001
- added link hand_rotation_v13_4, mass 0.49875676728406393; collision mesh filename=../meshes/hand_rotation_v13_4.stl scale=0.001 0.001 0.001; visual mesh filename=../meshes/hand_rotation_v13_4.stl scale=0.001 0.001 0.001
- added link hand_v17_1, mass 0.8585184504197826; collision mesh filename=../meshes/hand_v17_1.stl scale=0.001 0.001 0.001; visual mesh filename=../meshes/hand_v17_1.stl scale=0.001 0.001 0.001
- added link servo_holder2_v9_1, mass 0.4815312282713089; collision mesh filename=../meshes/servo_holder2_v9_1.stl scale=0.001 0.001 0.001; visual mesh filename=../meshes/servo_holder2_v9_1.stl scale=0.001 0.001 0.001
- added link servo_holder_v23_3, mass 0.39894172696668956; collision mesh filename=../meshes/servo_holder_v23_3.stl scale=0.001 0.001 0.001; visual mesh filename=../meshes/servo_holder_v23_3.stl scale=0.001 0.001 0.001
- link base_link: mass 0.8833573620888653 -> 0.3900830776668987
Joints:
- added joint Revolute 12: type continuous, parent base_link, child base_mount_v2_1, origin xyz=-0.00135 0.0369 -0.0165 rpy=0 0 0, axis 0.0 -0.0 -1.0
- joint Revolute 11: child servo_holder_v15_3 -> servo_holder_v23_3; origin xyz=0.0227 0.0 0.0125 rpy=0 0 0 -> xyz=0.02255 -0.0369 0.029 rpy=0 0 0; parent base_link -> base_mount_v2_1
- joint Revolute 7: axis -1.0 0.0 0.0 -> 1.0 -0.0 0.0; child servo_holder2_v2_1 -> servo_holder2_v9_1; origin xyz=0.0 0.1264 0.02945 rpy=0 0 0 -> xyz=0.0005 0.0324 0.02945 rpy=0 0 0; parent servo_holder_v15_3 -> servo_holder_v23_3
- joint Revolute 8: axis 1.0 -0.0 -0.0 -> 1.0 0.0 0.0; child hand_rotation_v11_4 -> hand_rotation_v13_4; origin xyz=0.0 0.1312 0.0 rpy=0 0 0 -> xyz=0.001 -0.0662 0.0 rpy=0 0 0; parent servo_holder2_v2_1 -> servo_holder2_v9_1
- joint Revolute 9: axis -0.0 -1.0 -0.0 -> -0.0 1.0 0.0; child hand_v15_1 -> hand_v17_1; origin xyz=-0.0232 0.0604 0.0 rpy=0 0 0 -> xyz=-0.0232 -0.0554 0.0 rpy=0 0 0; parent hand_rotation_v11_4 -> hand_rotation_v13_4

Commit message: Added joint constraint

File: urdf/arm_main.xacro (robot description, xacro)
@@ -123,15 +123,17 @@
   </collision>
 </link>
-<joint name="Revolute 7" type="continuous">
+<joint name="Revolute 7" type="revolute">
   <origin xyz="0.0005 0.0324 0.02945" rpy="0 0 0"/>
   <parent link="servo_holder_v23_3"/>
   <child link="servo_holder2_v9_1"/>
   <axis xyz="1.0 -0.0 0.0"/>
+  <limit upper="0.0" lower="-3.141593" effort="100" velocity="100"/>
 </joint>
-<joint name="Revolute 8" type="continuous">
+<joint name="Revolute 8" type="revolute">
   <origin xyz="0.001 -0.0662 0.0" rpy="0 0 0"/>
   <parent link="servo_holder2_v9_1"/>
   <child link="hand_rotation_v13_4"/>
   <axis xyz="1.0 0.0 0.0"/>
+  <limit upper="1.570796" lower="-0.349066" effort="100" velocity="100"/>
 </joint>
 <joint name="Revolute 9" type="continuous">
@@ -141,15 +143,17 @@
   <axis xyz="-0.0 1.0 0.0"/>
 </joint>
-<joint name="Revolute 11" type="continuous">
+<joint name="Revolute 11" type="revolute">
   <origin xyz="0.02255 -0.0369 0.029" rpy="0 0 0"/>
   <parent link="base_mount_v2_1"/>
   <child link="servo_holder_v23_3"/>
   <axis xyz="-1.0 -0.0 -0.0"/>
+  <limit upper="0.0" lower="-3.141593" effort="100" velocity="100"/>
 </joint>
-<joint name="Revolute 12" type="continuous">
+<joint name="Revolute 12" type="revolute">
   <origin xyz="-0.00135 0.0369 -0.0165" rpy="0 0 0"/>
   <parent link="base_link"/>
   <child link="base_mount_v2_1"/>
   <axis xyz="0.0 -0.0 -1.0"/>
+  <limit upper="1.570796" lower="-1.570796" effort="100" velocity="100"/>
 </joint>
 </robot>

File: urdf/komarm.urdf (robot description, URDF)
Before this commit: robot arm_main, 6 links, 5 joints
Joints:
- joint Revolute 11: limit (none) -> lower=-3.141593 upper=0.0 effort=100 velocity=100; type continuous -> revolute
- joint Revolute 12: limit (none) -> lower=-1.570796 upper=1.570796 effort=100 velocity=100; type continuous -> revolute
- joint Revolute 7: limit (none) -> lower=-3.141593 upper=0.0 effort=100 velocity=100; type continuous -> revolute
- joint Revolute 8: limit (none) -> lower=-0.349066 upper=1.570796 effort=100 velocity=100; type continuous -> revolute
