Commit message: update urdf file

File: robots/komarm/urdf/komarm.urdf (robot description, URDF)
Before this commit: robot arm_main, 6 links, 5 joints
Links:
- removed link base_mount_v2_1
- removed link hand_rotation_v13_4
- removed link hand_v17_1
- removed link servo_holder2_v9_1
- removed link servo_holder_v23_3
- added link arm_bracket_v1_2, mass 0.1366047605450555; collision mesh filename=../meshes/arm_bracket_v1_2.stl scale=0.001 0.001 0.001; visual mesh filename=../meshes/arm_bracket_v1_2.stl scale=0.001 0.001 0.001
- added link assembly_classis_v1_1, mass 10.00; collision mesh filename=../meshes/assembly_classis_v1_1.stl scale=0.001 0.001 0.001; visual mesh filename=../meshes/assembly_classis_v1_1.stl scale=0.001 0.001 0.001
- added link base_mount_v1_1, mass 0.4932742844219664; collision mesh filename=../meshes/base_mount_v1_1.stl scale=0.001 0.001 0.001; visual mesh filename=../meshes/base_mount_v1_1.stl scale=0.001 0.001 0.001
- added link hand_rotation_v1_4, mass 0.49875676728406393; collision mesh filename=../meshes/hand_rotation_v1_4.stl scale=0.001 0.001 0.001; visual mesh filename=../meshes/hand_rotation_v1_4.stl scale=0.001 0.001 0.001
- added link hand_v1_1, mass 0.8585184504197826; collision mesh filename=../meshes/hand_v1_1.stl scale=0.001 0.001 0.001; visual mesh filename=../meshes/hand_v1_1.stl scale=0.001 0.001 0.001
- added link servo_holder2_v1_1, mass 0.4815312282713089; collision mesh filename=../meshes/servo_holder2_v1_1.stl scale=0.001 0.001 0.001; visual mesh filename=../meshes/servo_holder2_v1_1.stl scale=0.001 0.001 0.001
- added link servo_holder_v1_3, mass 0.39894172696668956; collision mesh filename=../meshes/servo_holder_v1_3.stl scale=0.001 0.001 0.001; visual mesh filename=../meshes/servo_holder_v1_3.stl scale=0.001 0.001 0.001
Joints:
- added joint Rigid 13: type fixed, parent base_link, child arm_bracket_v1_2, origin xyz=-0.00135 0.0781 -0.02955 rpy=0 0 0
- added joint Rigid 14: type fixed, parent arm_bracket_v1_2, child assembly_classis_v1_1, origin xyz=-0.01 0.017 -0.0325 rpy=0 0 0
- joint Revolute 11: child servo_holder_v23_3 -> servo_holder_v1_3; parent base_mount_v2_1 -> base_mount_v1_1
- joint Revolute 12: child base_mount_v2_1 -> base_mount_v1_1
- joint Revolute 7: child servo_holder2_v9_1 -> servo_holder2_v1_1; parent servo_holder_v23_3 -> servo_holder_v1_3
- joint Revolute 8: child hand_rotation_v13_4 -> hand_rotation_v1_4; parent servo_holder2_v9_1 -> servo_holder2_v1_1
- joint Revolute 9: child hand_v17_1 -> hand_v1_1; parent hand_rotation_v13_4 -> hand_rotation_v1_4

File: robots/komarm/urdf/materials.xacro (robot description, xacro)
@@ -1,4 +1,4 @@
 <?xml version="1.0" ?>
-<robot name="arm_main" xmlns:xacro="http://www.ros.org/wiki/xacro" >
+<robot name="simulation" xmlns:xacro="http://www.ros.org/wiki/xacro" >
 <material name="silver_default">
   <color rgba="0.700 0.700 0.700 1.000"/>
@@ -7,3 +7,6 @@
   <color rgba="0.6274509803921569 0.6274509803921569 0.6274509803921569 1.0"/>
 </material>
+<material name="aluminum_satin">
+  <color rgba="0.9607843137254902 0.9607843137254902 0.9647058823529412 1.0"/>
+</material>
 </robot>

Commit message: update urdf

File: robots/komarm/urdf/komarm.urdf (robot description, URDF)
Before this commit: robot simulation, 8 links, 7 joints
Links:
- removed link arm_bracket_v1_2
- removed link assembly_classis_v1_1
- removed link base_mount_v1_1
- removed link hand_rotation_v1_4
- removed link hand_v1_1
- removed link servo_holder2_v1_1
- removed link servo_holder_v1_3
- added link hand_finger_v1_1, mass 0.18407843738656002; collision mesh filename=../meshes/hand_finger_v1_1.stl scale=0.001 0.001 0.001; visual mesh filename=../meshes/hand_finger_v1_1.stl scale=0.001 0.001 0.001
- added link hand_unit_v1_1, mass 0.6163609537224307; collision mesh filename=../meshes/hand_unit_v1_1.stl scale=0.001 0.001 0.001; visual mesh filename=../meshes/hand_unit_v1_1.stl scale=0.001 0.001 0.001
- added link pitch_1_test_v5_1, mass 0.5173712582672985; collision mesh filename=../meshes/pitch_1_test_v5_1.stl scale=0.001 0.001 0.001; visual mesh filename=../meshes/pitch_1_test_v5_1.stl scale=0.001 0.001 0.001
- added link pitch_2_test_v1_1, mass 0.4049688490988578; collision mesh filename=../meshes/pitch_2_test_v1_1.stl scale=0.001 0.001 0.001; visual mesh filename=../meshes/pitch_2_test_v1_1.stl scale=0.001 0.001 0.001
- added link roll_1_test_v11_1, mass 0.45569427768407117; collision mesh filename=../meshes/roll_1_test_v11_1.stl scale=0.001 0.001 0.001; visual mesh filename=../meshes/roll_1_test_v11_1.stl scale=0.001 0.001 0.001
- added link roll_2_test_v1_1, mass 0.45660397486942944; collision mesh filename=../meshes/roll_2_test_v1_1.stl scale=0.001 0.001 0.001; visual mesh filename=../meshes/roll_2_test_v1_1.stl scale=0.001 0.001 0.001
- link base_link: mass 0.3900830776668987 -> 0.3893898243402566
Joints:
- removed joint Revolute 11
- removed joint Revolute 12
- removed joint Revolute 7
- removed joint Revolute 8
- removed joint Revolute 9
- removed joint Rigid 13
- removed joint Rigid 14
- added joint Revolute 1: type revolute, parent base_link, child pitch_1_test_v5_1, origin xyz=0.00035 -0.0369 0.0062 rpy=0 0 0, axis 0.0 0.0 -1.0, limit lower=-1.570796 upper=1.570796 effort=100 velocity=100
- added joint Revolute 2: type revolute, parent pitch_1_test_v5_1, child roll_1_test_v11_1, origin xyz=0.02035 0.0622 0.00545 rpy=0 0 0, axis -1.0 -0.0 -0.0, limit lower=-1.396263 upper=1.745329 effort=100 velocity=100
- added joint Revolute 3: type continuous, parent roll_1_test_v11_1, child pitch_2_test_v1_1, origin xyz=-0.0212 0.0564 0.0 rpy=0 0 0, axis -0.0 1.0 -0.0
- added joint Revolute 4: type revolute, parent pitch_2_test_v1_1, child roll_2_test_v1_1, origin xyz=0.021 0.0462 0.0 rpy=0 0 0, axis -1.0 0.0 -0.0, limit lower=-1.396263 upper=1.919862 effort=100 velocity=100
- added joint Revolute 5: type continuous, parent roll_2_test_v1_1, child hand_unit_v1_1, origin xyz=-0.0212 0.0564 0.0 rpy=0 0 0, axis 0.0 -1.0 -0.0
- added joint Revolute 6: type revolute, parent hand_unit_v1_1, child hand_finger_v1_1, origin xyz=0.0222 0.02565 0.013 rpy=0 0 0, axis -1.0 -0.0 0.0, limit lower=-1.047198 upper=0.872665 effort=100 velocity=100

File: robots/komarm/urdf/materials.xacro (robot description, xacro)
@@ -1,4 +1,4 @@
 <?xml version="1.0" ?>
-<robot name="simulation" xmlns:xacro="http://www.ros.org/wiki/xacro" >
+<robot name="arm_test_main" xmlns:xacro="http://www.ros.org/wiki/xacro" >
 <material name="silver_default">
   <color rgba="0.700 0.700 0.700 1.000"/>
@@ -7,6 +7,3 @@
   <color rgba="0.6274509803921569 0.6274509803921569 0.6274509803921569 1.0"/>
 </material>
-<material name="aluminum_satin">
-  <color rgba="0.9607843137254902 0.9607843137254902 0.9647058823529412 1.0"/>
-</material>
 </robot>
